Commit message: finally got 0.2 working

File: robot_description/urdf/mobile_manipulator.urdf (robot description, URDF)
Before this commit: robot mobile_manipulator, 10 links, 9 joints
Links:
- removed link front_left_wheel
- removed link front_right_wheel
- removed link rear_left_wheel
- removed link rear_right_wheel
- added link wheel_left_link, mass 2.8498940e-02; collision cylinder length=0.018 radius=0.033; visual mesh filename=package://turtlebot3_description/meshes/wheels/left_tire.stl scale=0.002 0.002 0.002
- added link wheel_right_link, mass 2.8498940e-02; collision cylinder length=0.018 radius=0.033; visual mesh filename=package://turtlebot3_description/meshes/wheels/right_tire.s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 scale=0.002 0.002 0.002
- link base_link: mass 47.873 -> 1.3729096e+00; geometry collision box size=0.266 0.266 0.094; visual mesh filename=package://turtlebot3_description/meshes/bases/waffle_base.s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 scale=0.002 0.002 0.002
Joints:
- removed joint front_left_wheel_joint
- removed joint front_right_wheel_joint
- removed joint rear_left_wheel_joint
- removed joint rear_right_wheel_joint
- added joint wheel_left_joint: type continuous, parent base_link, child wheel_left_link, origin xyz=0.0 0.144 0.023 rpy=-1.57 0 0, axis 0 0 1
- added joint wheel_right_joint: type continuous, parent base_link, child wheel_right_link, origin xyz=0.0 -0.144 0.023 rpy=-1.57 0 0, axis 0 0 1
- joint arm_base_joint: axis 0 0 1 -> 0 0 0.5; origin xyz=0.20 0.0 0.145 rpy=0 0 0 -> xyz=-0.1 0.0 0.18 rpy=0 0 0

File: robot_description/urdf/mobile_manipulator.urdf.xacro (robot description, xacro)
@@ -1,6 +1,6 @@
 <?xml version="1.0"?>
-<robot xmlns:xacro="http://ros.org/wiki/xacro" name="robot_base" >
-<xacro:include filename="$(find robot_description)/urdf/robot_base.urdf.xacro" />
-<xacro:include filename="$(find robot_description)/urdf/robot_arm.urdf.xacro" />
-<xacro:arm_joint prefix="arm_base_link" parent="base_link" child="arm_base" originxyz="0.20 0.0 0.145" originrpy="0 0 0"/>
+<robot xmlns:xacro="http://ros.org/wiki/xacro" name="robot_base">
+    <xacro:include filename="$(find robot_description)/urdf/robot_base.urdf.xacro" />
+    <xacro:include filename="$(find robot_description)/urdf/robot_arm.urdf.xacro" />
+    <xacro:arm_joint prefix="arm_base_link" parent="base_link" child="arm_base" originxyz="0.20 0.0 0.145" originrpy="0 0 0" />
 </robot>
